File: Kicad/robik2.kicad_pcb (KiCad board)
At the start: 2 copper layers, 13 parts, among them J1 Conn_01x06_Male, J2 Conn_01x06_Male, J3 Conn_01x08_Male, J4 Conn_01x08_Male, J5 Conn_01x03_Male, Q1 BUZ11, U1 LM7805_TO220

Commit message: board
Parts:
- added C3: CP, Capacitor_THT:CP_Radial_D5.0mm_P2.00mm, F.Cu at (53.2, 63.2)
- added C4: CP, Capacitor_THT:CP_Radial_D5.0mm_P2.00mm, F.Cu at (53.2, 68.9)
- added C5: CP, Capacitor_THT:CP_Radial_D5.0mm_P2.00mm, F.Cu at (53.2, 57.5)
- added D3: 1N4007, Diode_THT:D_A-405_P10.16mm_Horizontal, F.Cu at (68.8, 63.5)
- added F2: Pojistka 2A, Fuse:Fuse_sbeve, F.Cu at (61.0, 70.2)
- added J6: Servo, Connector_PinHeader_2.00mm:PinHeader_1x03_P2.00mm_Vertical, F.Cu at (93.0, 69.5)
- added J7: Ultrasound 2, Connector_PinHeader_2.00mm:PinHeader_1x05_P2.00mm_Vertical, F.Cu at (80.5, 85.0)
- added J8: Motor terminal, TerminalBlock:TerminalBlock_bornier-2_P5.08mm, F.Cu at (63.2, 46.2)
- added J9: Battery terminal, TerminalBlock:TerminalBlock_bornier-2_P5.08mm, F.Cu at (52.8, 46.2)
- added R1: R, Resistor_THT:R_Axial_DIN0207_L6.3mm_D2.5mm_P10.16mm_Horizontal, F.Cu at (97.0, 24.2)
- added R2: R, Resistor_THT:R_Axial_DIN0207_L6.3mm_D2.5mm_P7.62mm_Horizontal, F.Cu at (97.8, 92.5)
- added R3: R, Resistor_THT:R_Axial_DIN0207_L6.3mm_D2.5mm_P10.16mm_Horizontal, F.Cu at (119.5, 94.5)
- added SW1: Greenbtn, Button_Switch_THT:SW_PUSH-12mm, F.Cu at (78.0, 92.2)
- added SW2: Resetbtn, Button_Switch_THT:SW_PUSH_6mm, F.Cu at (61.5, 85.8)
- added SW3: Ebtn, Button_Switch_THT:SW_PUSH_6mm, F.Cu at (66.0, 98.5)
- added SW4: Redbtn, Button_Switch_THT:SW_PUSH-12mm, F.Cu at (91.0, 92.2)
- F1: footprint Fuse:Fuseholder_Cylinder-5x20mm_Schurter_0031_8201_Horizontal_Open -> Fuse:Fuse_sbeve
- J1: value Conn_01x06_Male -> Analog 0-5; moved to B.Cu
- J2: value Conn_01x06_Male -> Power and other; footprint Connector_PinSocket_2.00mm:PinSocket_1x06_P2.00mm_Vertical_SMD_Pin1Left -> Connector_PinSocket_2.00mm:PinSocket_1x08_P2.00mm_Vertical_SMD_Pin1Left; moved to B.Cu
- J3: value Conn_01x08_Male -> Digital 0-7; moved to B.Cu
- J4: value Conn_01x08_Male -> Digital 8-13; moved to B.Cu
- J5: value Conn_01x03_Male -> Ultrasound 1; footprint Connector_PinSocket_2.00mm:PinSocket_1x03_P2.00mm_Vertical -> Connector_PinHeader_2.00mm:PinHeader_1x05_P2.00mm_Vertical
- RV1: footprint Potentiometer_THT:Potentiometer_ACP_CA14V-15_Vertical -> Potentiometer_THT:Potentiometer_Runtron_RM-065_Vertical
- moved J3 64.8 mm to (104.0, 97.8)
- moved F1 63.0 mm to (103.5, 60.0), turned to 180 degrees
- moved J1 61.8 mm to (55.0, 99.8)
- moved D1 58.7 mm to (115.2, 97.2)
- moved C1 55.6 mm to (95.8, 49.8)
- moved C2 51.4 mm to (100.8, 52.8), turned to 180 degrees
- moved J2 50.5 mm to (55.0, 82.8)
- moved D2 50.2 mm to (97.8, 105.2), turned to 90 degrees
- moved J4 47.9 mm to (104.0, 79.8)
- moved RV1 42.9 mm to (61.5, 95.2), turned to 90 degrees
- moved J5 40.4 mm to (84.5, 77.0), turned to 90 degrees
- moved U1 18.5 mm to (97.5, 45.0)
- moved Q1 15.4 mm to (79.0, 45.5)
Connections:
- C1 pad 1: Net-(C1-Pad1) -> +7.5V
- C1 pad 2: Net-(C1-Pad2) -> GND
- C2 pad 1: Net-(C2-Pad1) -> +5V
- C2 pad 2: Net-(C2-Pad2) -> GND
- D1 pad 1: Net-(D1-Pad1) -> GND
- D2 pad 1: Net-(D2-Pad1) -> GND
- F1 pad 1: Net-(F1-Pad1) -> +5V
- J2 pad 1: Net-(J2-Pad1) -> +7.5V
- J2 pad 2: Net-(J2-Pad2) -> GND
- J2 pad 3: Net-(J2-Pad3) -> GND
- J2 pad 4: Net-(J2-Pad4) -> +5VA
- J5 pad 1: Net-(J5-Pad1) -> GND
- J5 pad 3: Net-(J5-Pad3) -> Net-(J3-Pad8)
- Q1 pad 1: Net-(Q1-Pad1) -> Net-(J4-Pad4)
- Q1 pad 3: Net-(Q1-Pad3) -> GND
- RV1 pad 1: Net-(RV1-Pad1) -> GND
- RV1 pad 2: Net-(RV1-Pad2) -> Net-(J1-Pad1)
- RV1 pad 3: Net-(RV1-Pad3) -> +5VA
- U1 pad 1: Net-(U1-Pad1) -> +7.5V
- U1 pad 2: Net-(U1-Pad2) -> GND
- U1 pad 3: Net-(U1-Pad3) -> +5V
Routing:
- net GND: track 0.00 -> 173.6 mm
- net Net-(J3-Pad5): track 0.00 -> 41.1 mm
- net +7.5V: track 0.00 -> 35.6 mm
- net Net-(J3-Pad4): track 0.00 -> 31.7 mm
- net Net-(J1-Pad1): track 0.00 -> 24.1 mm
- net Net-(J3-Pad3): track 0.00 -> 16.5 mm
- net +5VA: track 0.00 -> 9.35 mm
- net Net-(J3-Pad6): track 0.00 -> 8.78 mm
- net Net-(J2-Pad6): track 0.00 -> 5.11 mm
- net Net-(D2-Pad2): track 0.00 -> 2.59 mm
- net Net-(J4-Pad1): track 0.00 -> 1.30 mm
- net Net-(F1-Pad2): track 0.00 -> 0.71 mm
- net +5V: track 0.00 -> 0.67 mm
